File: Modulo_PT2313L/_autosave-Modulo_PT2313L.kicad_pcb (KiCad board)
At the start: 2 copper layers, 100 x 50 mm, 40 parts, among them J1 Power 9V, J2 LF_Amp, J3 RF_Amp, J4 LR_Amp, J5 RR_Amp, J6 I2C_Conn, J7 Inputs, U1 PT2313

Commit message: agrego imagenes y esquematico
Other:
- board text added: "+"
- board text added: "-"
- board text added: "1->"
- board text added: "1-LIN1 2-LIN2 3-LIN3 4-RIN1 5-RIN3 6-RIN2"
- board text added: "9-12V"
- board text added: "Diseñado por Emanuel Decima Procesador de Audio de 4 Canales Basado en IC PT2313L"
- board text added: "Gnd"
- board text added: "LF-Amp"
- board text added: "LR-Amp"
- board text added: "RR-Amp"
- board text added: "SCL"
- board text added: "SDA"
- board text added: "Vcc"
Changed lines of the file:
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@@
 		)
+	)
+	(gr_line
+		(start 162.72 87.02)
+		(end 164.76 85.04)
+		(stroke
+			(width 0.1)
+			(type default)
+		)
+		(layer "F.SilkS")
+	)
+	(gr_line
+		(start 156.3 87.02)
+		(end 162.72 87.02)
+		(stroke
+			(width 0.1)
+			(type default)
+		)
+		(layer "F.SilkS")
 	)
 	(gr_arc
@@
 		(layer "Edge.Cuts")
 	)
+	(gr_text "LR-Amp"
+		(at 80.83 70.31 0)
+		(layer "F.SilkS")
+		(effects
+			(font
+				(size 1 1)
+				(thickness 0.1)
+			)
+			(justify left bottom)
+		)
+	)
+	(gr_text "9-12V"
+		(at 165.2 43.33 0)
+		(layer "F.SilkS")
+		(effects
+			(font
+				(size 1 1)
+				(thickness 0.1)
+			)
+			(justify left bottom)
+		)
+	)
+	(gr_text "SCL\n"
+		(at 126.57 48.55 0)
+		(layer "F.SilkS")
+		(effects
+			(font
+				(size 1 0.5)
+				(thickness 0.1)
+			)
+			(justify left bottom)
+		)
+	)
+	(gr_text "1->"
+		(at 133.69 88.55 0)
+		(layer "F.SilkS")
+		(effects
+			(font
+				(size 1 1)
+				(thickness 0.1)
+			)
+			(justify left bottom)
+		)
+	)
+	(gr_text "LF-Amp"
+		(at 80.87 59.06 0)
+		(layer "F.SilkS")
+		(effects
+			(font
+				(size 1 1)
+				(thickness 0.1)
+			)
+			(justify left bottom)
+		)
+	)
+	(gr_text "SDA"
+		(at 126.558096 51.163333 0)
+		(layer "F.SilkS")
+		(effects
+			(font
+				(size 1 0.5)
+				(thickness 0.1)
+			)
+			(justify left bottom)
+		)
+	)
+	(gr_text "RR-Amp"
+		(at 80.61 81.64 0)
+		(layer "F.SilkS")
+		(effects
+			(font
+				(size 1 1)
+				(thickness 0.1)
+			)
+			(justify left bottom)
+		)
+	)
+	(gr_text "-"
+		(at 152.92 41.77 0)
+		(layer "F.SilkS")
+		(effects
+			(font
+				(size 1 1)
+				(thickness 0.1)
+			)
+			(justify left bottom)
+		)
+	)
+	(gr_text "LF-Amp"
+		(at 80.77 49.64 0)
+		(layer "F.SilkS")
+		(effects
+			(font
+				(size 1 1)
+				(thickness 0.1)
+			)
+			(justify left bottom)
+		)
+	)
+	(gr_text "+"
+		(at 165.01 41.83 0)
+		(layer "F.SilkS")
+		(effects
+			(font
+				(size 1 1)
+				(thickness 0.1)
+			)
+			(justify left bottom)
+		)
+	)
+	(gr_text "Gnd"
+		(at 126.558095 53.776667 0)
+		(layer "F.SilkS")
+		(effects
+			(font
+				(size 1 0.5)
+				(thickness 0.1)
+			)
+			(justify left bottom)
+		)
+	)
+	(gr_text "Diseñado por Emanuel Decima\n\nProcesador de Audio de 4 Canales\nBasado en IC PT2313L"
+		(at 102.89 87.09 0)
+		(layer "F.SilkS")
+		(effects
+			(font
+				(size 1 1)
+				(thickness 0.2)
+				(bold yes)
+			)
+			(justify left bottom)
+		)
+	)
+	(gr_text "1-LIN1\n2-LIN2\n3-LIN3\n4-RIN1\n5-RIN3\n6-RIN2"
+		(at 165.78 86.36 0)
+		(layer "F.SilkS")
+		(effects
+			(font
+				(size 1 1)
+				(thickness 0.1)
+			)
+			(justify left bottom)
+		)
+	)
+	(gr_text "Vcc"
+		(at 126.61762 56.39 0)
+		(layer "F.SilkS")
+		(effects
+			(font
+				(size 1 0.5)
+				(thickness 0.1)
+			)
+			(justify left bottom)
+		)
+	)
 	(segment
